Commit message: Improvements for simulation

File: zed_wrapper/urdf/zed_descr.urdf.xacro (robot description, xacro)
@@ -16,4 +16,5 @@
 -->
 <robot name="stereolabs_camera" xmlns:xacro="http://ros.org/wiki/xacro">
+  <link name="$(arg base_frame)" />
   <xacro:arg name="camera_name"   default="zed" />
   <xacro:arg name="camera_model"  default="zed" />
@@ -29,4 +30,3 @@
     <origin xyz="$(arg cam_pos_x) $(arg cam_pos_y) $(arg cam_pos_z)" rpy="$(arg cam_roll) $(arg cam_pitch) $(arg cam_yaw)" />
   </xacro:zed_camera>
-  <link name="$(arg base_frame)" />
 </robot>

Commit message: Change STL load behavior

File: zed_wrapper/urdf/zed_descr.urdf.xacro (robot description, xacro)
@@ -26,6 +26,7 @@
   <xacro:arg name="cam_pitch"     default="0.0" />
   <xacro:arg name="cam_yaw"       default="0.0" />
+  <xacro:arg name="mesh_file"     default="" />
   <xacro:include filename="$(find zed_wrapper)/urdf/zed_macro.urdf.xacro" />
-  <xacro:zed_camera name="$(arg camera_name)" model="$(arg camera_model)" parent="$(arg base_frame)">
+  <xacro:zed_camera name="$(arg camera_name)" model="$(arg camera_model)" parent="$(arg base_frame)" mesh_file="$(arg mesh_file)">
     <origin xyz="$(arg cam_pos_x) $(arg cam_pos_y) $(arg cam_pos_z)" rpy="$(arg cam_roll) $(arg cam_pitch) $(arg cam_yaw)" />
   </xacro:zed_camera>

File: zed_wrapper/urdf/zed_macro.urdf.xacro (robot description, xacro)
@@ -16,7 +16,7 @@
 -->
 <robot xmlns:xacro="http://wiki.ros.org/xacro">
-	<xacro:include filename="$(find zed_wrapper)/urdf/include/materials.urdf.xacro" />
-	<xacro:property name="M_PI" value="3.1415926535897931" />
-	<!--
+  <xacro:include filename="$(find zed_wrapper)/urdf/include/materials.urdf.xacro" />
+  <xacro:property name="M_PI"     value="3.1415926535897931" />
+  <!--
     Parameters:
       - name: the camera's name.  should match the parameter sent to the launch file for this camera
@@ -25,117 +25,119 @@
       - origin: the xyz/rpy offset from the parent link
   -->
-	<xacro:macro name="zed_camera" params="name=zed model=zed parent *origin">
-		<xacro:if value="${model == 'zed'}">
-			<xacro:property name="baseline" value="0.12" />
-			<xacro:property name="height" value="0.03" />
-			<xacro:property name="bottom_slope" value="0.05" />
-			<xacro:property name="screw_offset_x" value="0.0" />
-			<xacro:property name="optical_offset_x" value="-0.01" />
-		</xacro:if>
-		<xacro:if value="${model == 'zedm'}">
-			<xacro:property name="baseline" value="0.06" />
-			<xacro:property name="height" value="0.0265" />
-			<xacro:property name="bottom_slope" value="0.0" />
-			<xacro:property name="screw_offset_x" value="0.0" />
-			<xacro:property name="optical_offset_x" value="0.0" />
-		</xacro:if>
-		<xacro:if value="${model == 'zed2'}">
-			<xacro:property name="baseline" value="0.12" />
-			<xacro:property name="height" value="0.03" />
-			<xacro:property name="bottom_slope" value="0.05" />
-			<xacro:property name="screw_offset_x" value="0.0" />
-			<xacro:property name="optical_offset_x" value="-0.01" />
-		</xacro:if>
-		<xacro:if value="${model == 'zed2i'}">
-			<xacro:property name="baseline" value="0.12" />
-			<xacro:property name="height" value="0.03" />
-			<xacro:property name="bottom_slope" value="0.0" />
-			<xacro:property name="screw_offset_x" value="-0.01" />
-			<xacro:property name="optical_offset_x" value="-0.01" />
-		</xacro:if>
-		<!-- Camera mounting point (the threaded screw hole in the bottom) -->
-		<link name="${name}_base_link">
-			<visual>
-				<origin xyz="${screw_offset_x} 0 ${height/2}" rpy="0 0 0"/>
-				<geometry>
-					<mesh filename="package://zed_interfaces/meshes/${model}.stl" />
-				</geometry>
-				<material name="${model}_mat" />
-			</visual>
-			<collision>
-				<geometry>
-					<mesh filename="package://zed_interfaces/meshes/${model}.stl" />
-				</geometry>
-			</collision>
-			<inertial>
-				<mass value="0.125" />
-				<inertia ixx="0.000028521" ixy="0.0" ixz="0.0" iyy="0.000465434" iyz="0.0" izz="0.000468458"/>
-			</inertial>
-		</link>
-		<joint name="${name}_base_joint" type="fixed">
-			<parent link="${parent}"/>
-			<child link="${name}_base_link"/>
-			<xacro:insert_block name="origin" />
-		</joint>
-		<!-- Camera Center -->
-		<link name="${name}_camera_center" />
-		<joint name="${name}_camera_center_joint" type="fixed">
-			<parent link="${name}_base_link"/>
-			<child link="${name}_camera_center"/>
-			<origin xyz="0 0 ${height/2}" rpy="0 ${bottom_slope} 0" />
-		</joint>
-		<!-- Left Camera -->
-		<link name="${name}_left_camera_frame" />
-		<joint name="${name}_left_camera_joint" type="fixed">
-			<parent link="${name}_camera_center"/>
-			<child link="${name}_left_camera_frame"/>
-			<origin xyz="0 ${baseline/2} 0" rpy="0 0 0" />
-		</joint>
-		<link name="${name}_left_camera_optical_frame"/>
-		<joint name="${name}_left_camera_optical_joint" type="fixed">
-			<origin xyz="${optical_offset_x} 0 0" rpy="-${M_PI/2} 0.0 -${M_PI/2}"/>
-			<parent link="${name}_left_camera_frame"/>
-			<child link="${name}_left_camera_optical_frame"/>
-		</joint>
-		<!-- Right Camera -->
-		<link name="${name}_right_camera_frame" />
-		<joint name="${name}_right_camera_joint" type="fixed">
-			<parent link="${name}_camera_center"/>
-			<child link="${name}_right_camera_frame"/>
-			<origin xyz="0 -${baseline/2} 0" rpy="0 0 0" />
-		</joint>
-		<link name="${name}_right_camera_optical_frame"/>
-		<joint name="${name}_right_camera_optical_joint" type="fixed">
-			<origin xyz="${optical_offset_x} 0 0" rpy="-${M_PI/2} 0.0 -${M_PI/2}"/>
-			<parent link="${name}_right_camera_frame"/>
-			<child link="${name}_right_camera_optical_frame"/>
-		</joint>
-		<!-- ZED2 Sensors -->
-		<xacro:if value="${model == 'zed2' or model == 'zed2i'}">
-			<link name="${name}_mag_link" />
-			<joint name="${name}_mag_joint" type="fixed">
-				<parent link="${name}_camera_center"/>
-				<child link="${name}_mag_link"/>
-				<origin xyz="0 0 0" rpy="0 0 0" />
-			</joint>
-			<link name="${name}_baro_link" />
-			<joint name="${name}_baro_joint" type="fixed">
-				<parent link="${name}_camera_center"/>
-				<child link="${name}_baro_link"/>
-				<origin xyz="0 0 0" rpy="0 0 0" />
-			</joint>
-			<link name="${name}_temp_left_link" />
-			<joint name="${name}_temp_left_joint" type="fixed">
-				<parent link="${name}_left_camera_frame"/>
-				<child link="${name}_temp_left_link"/>
-				<origin xyz="0 0 0" rpy="0 0 0" />
-			</joint>
-			<link name="${name}_temp_right_link" />
-			<joint name="${name}_temp_right_joint" type="fixed">
-				<parent link="${name}_right_camera_frame"/>
-				<child link="${name}_temp_right_link"/>
-				<origin xyz="0 0 0" rpy="0 0 0" />
-			</joint>
-		</xacro:if>
-	</xacro:macro>
+  <xacro:macro name="zed_camera" params="name=zed model=zed parent mesh_file *origin">
+    <xacro:if value="${model == 'zed'}">
+      <xacro:property name="baseline" value="0.12" />
+      <xacro:property name="height" value="0.03" />
+      <xacro:property name="bottom_slope" value="0.05" />
+      <xacro:property name="screw_offset_x" value="0.0" />
+      <xacro:property name="optical_offset_x" value="-0.01" />
+    </xacro:if>
+    <xacro:if value="${model == 'zedm'}">
+      <xacro:property name="baseline" value="0.06" />
+      <xacro:property name="height" value="0.0265" />
+      <xacro:property name="bottom_slope" value="0.0" />
+      <xacro:property name="screw_offset_x" value="0.0" />
+      <xacro:property name="optical_offset_x" value="0.0" />
+    </xacro:if>
+    <xacro:if value="${model == 'zed2'}">
+      <xacro:property name="baseline" value="0.12" />
+      <xacro:property name="height" value="0.03" />
+      <xacro:property name="bottom_slope" value="0.05" />
+      <xacro:property name="screw_offset_x" value="0.0" />
+      <xacro:property name="optical_offset_x" value="-0.01" />
+    </xacro:if>
+    <xacro:if value="${model == 'zed2i'}">
+      <xacro:property name="baseline" value="0.12" />
+      <xacro:property name="height" value="0.03" />
+      <xacro:property name="bottom_slope" value="0.0" />
+      <xacro:property name="screw_offset_x" value="-0.01" />
+      <xacro:property name="optical_offset_x" value="-0.01" />
+    </xacro:if>
+    <!-- Camera mounting point (the threaded screw hole in the bottom) -->
+    <link name="${name}_base_link">
+      <visual>
+	      <origin xyz="${screw_offset_x} 0 ${height/2}" rpy="0 0 0"/>
+	      <geometry>
+		      <!-- <mesh filename="package://zed_interfaces/meshes/${model}.stl" /> -->
+          <mesh filename="file://${mesh_file}" />
+	      </geometry>
+	      <material name="${model}_mat" />
+      </visual>
+      <collision>
+        <geometry>
+          <!-- <mesh filename="package://zed_interfaces/meshes/${model}.stl" /> -->
+          <mesh filename="file://${mesh_file}" />
+        </geometry>
+      </collision>
+      <inertial>
+        <mass value="0.125" />
+        <inertia ixx="0.000028521" ixy="0.0" ixz="0.0" iyy="0.000465434" iyz="0.0" izz="0.000468458"/>
+      </inertial>
+    </link>
+    <joint name="${name}_base_joint" type="fixed">
+      <parent link="${parent}"/>
+      <child link="${name}_base_link"/>
+      <xacro:insert_block name="origin" />
+    </joint>
+    <!-- Camera Center -->
+    <link name="${name}_camera_center" />
+    <joint name="${name}_camera_center_joint" type="fixed">
+      <parent link="${name}_base_link"/>
+      <child link="${name}_camera_center"/>
+      <origin xyz="0 0 ${height/2}" rpy="0 ${bottom_slope} 0" />
+    </joint>
+    <!-- Left Camera -->
+    <link name="${name}_left_camera_frame" />
+    <joint name="${name}_left_camera_joint" type="fixed">
+      <parent link="${name}_camera_center"/>
+      <child link="${name}_left_camera_frame"/>
+      <origin xyz="0 ${baseline/2} 0" rpy="0 0 0" />
+    </joint>
+    <link name="${name}_left_camera_optical_frame"/>
+    <joint name="${name}_left_camera_optical_joint" type="fixed">
+      <origin xyz="${optical_offset_x} 0 0" rpy="-${M_PI/2} 0.0 -${M_PI/2}"/>
+      <parent link="${name}_left_camera_frame"/>
+      <child link="${name}_left_camera_optical_frame"/>
+    </joint>
+    <!-- Right Camera -->
+    <link name="${name}_right_camera_frame" />
+    <joint name="${name}_right_camera_joint" type="fixed">
+      <parent link="${name}_camera_center"/>
+      <child link="${name}_right_camera_frame"/>
+      <origin xyz="0 -${baseline/2} 0" rpy="0 0 0" />
+    </joint>
+    <link name="${name}_right_camera_optical_frame"/>
+    <joint name="${name}_right_camera_optical_joint" type="fixed">
+      <origin xyz="${optical_offset_x} 0 0" rpy="-${M_PI/2} 0.0 -${M_PI/2}"/>
+      <parent link="${name}_right_camera_frame"/>
+      <child link="${name}_right_camera_optical_frame"/>
+    </joint>
+    <!-- ZED2 Sensors -->
+    <xacro:if value="${model == 'zed2' or model == 'zed2i'}">
+      <link name="${name}_mag_link" />
+      <joint name="${name}_mag_joint" type="fixed">
+        <parent link="${name}_camera_center"/>
+        <child link="${name}_mag_link"/>
+        <origin xyz="0 0 0" rpy="0 0 0" />
+      </joint>
+      <link name="${name}_baro_link" />
+      <joint name="${name}_baro_joint" type="fixed">
+        <parent link="${name}_camera_center"/>
+        <child link="${name}_baro_link"/>
+        <origin xyz="0 0 0" rpy="0 0 0" />
+      </joint>
+      <link name="${name}_temp_left_link" />
+      <joint name="${name}_temp_left_joint" type="fixed">
+        <parent link="${name}_left_camera_frame"/>
+        <child link="${name}_temp_left_link"/>
+        <origin xyz="0 0 0" rpy="0 0 0" />
+      </joint>
+      <link name="${name}_temp_right_link" />
+      <joint name="${name}_temp_right_joint" type="fixed">
+        <parent link="${name}_right_camera_frame"/>
+        <child link="${name}_temp_right_link"/>
+        <origin xyz="0 0 0" rpy="0 0 0" />
+      </joint>
+    </xacro:if>
+  </xacro:macro>
 </robot>

Commit message: Fix for URDF in simulation

File: zed_wrapper/urdf/zed_descr.urdf.xacro (robot description, xacro)
@@ -16,18 +16,60 @@
 -->
 <robot name="stereolabs_camera" xmlns:xacro="http://ros.org/wiki/xacro">
-  <link name="$(arg base_frame)" />
-  <xacro:arg name="camera_name"   default="zed" />
-  <xacro:arg name="camera_model"  default="zed" />
-  <xacro:arg name="base_frame"    default="base_link" />
-  <xacro:arg name="cam_pos_x"     default="0.0" />
-  <xacro:arg name="cam_pos_y"     default="0.0" />
-  <xacro:arg name="cam_pos_z"     default="0.0" />
-  <xacro:arg name="cam_roll"      default="0.0" />
-  <xacro:arg name="cam_pitch"     default="0.0" />
-  <xacro:arg name="cam_yaw"       default="0.0" />
-  <xacro:arg name="mesh_file"     default="" />
+  <xacro:arg name="camera_name"     default="zed" />
+  <xacro:arg name="camera_model"    default="zed" />
+  <xacro:arg name="use_base_frame"  default="true" />
+  <xacro:arg name="base_frame"      default="base_link" />
+  <xacro:arg name="cam_pos_x"       default="0.0" />
+  <xacro:arg name="cam_pos_y"       default="0.0" />
+  <xacro:arg name="cam_pos_z"       default="0.0" />
+  <xacro:arg name="cam_roll"        default="0.0" />
+  <xacro:arg name="cam_pitch"       default="0.0" />
+  <xacro:arg name="cam_yaw"         default="0.0" />
+  <xacro:arg name="mesh_file"       default="" />
   <xacro:include filename="$(find zed_wrapper)/urdf/zed_macro.urdf.xacro" />
-  <xacro:zed_camera name="$(arg camera_name)" model="$(arg camera_model)" parent="$(arg base_frame)" mesh_file="$(arg mesh_file)">
+  <xacro:zed_camera name="$(arg camera_name)" model="$(arg camera_model)" declare_parent="$(arg use_base_frame)" parent="$(arg base_frame)" mesh_file="$(arg mesh_file)">
     <origin xyz="$(arg cam_pos_x) $(arg cam_pos_y) $(arg cam_pos_z)" rpy="$(arg cam_roll) $(arg cam_pitch) $(arg cam_yaw)" />
   </xacro:zed_camera>
+  <gazebo>
+    <!-- <plugin name="sl_simul::ZedSystem" filename="/home/walter/devel/Gazebo/build-zed-gazebo-Desktop_Qt_5_15_2_GCC_64bit-Release/zed_plugin/libZedIgnitionPlugin.so"> -->
+    <plugin name="sl_simul::ZedSystem" filename="ZedIgnitionPlugin">
+      <zed_model>zed</zed_model>
+      <zed_serial_number>510</zed_serial_number>
+      <zed_resolution>HD720</zed_resolution>
+      <zed_framerate>30</zed_framerate>
+      <zed_sim_idx>0</zed_sim_idx>
+    </plugin>
+  </gazebo>
+  <gazebo reference="$(arg camera_name)_base_link">
+      <sensor name="zed_left" type="camera">
+        <pose>0 0.06 0 0 0 0</pose>
+        <update_rate>30</update_rate>
+        <always_on>1</always_on>
+        <topic>zed/left</topic>
+        <camera>
+          <image>
+            <format>RGB_INT8</format>
+          </image>
+          <clip>
+            <near>0.01</near>
+            <far>3000</far>
+          </clip>
+        </camera>
+      </sensor>
+      <sensor name="zed_right" type="camera">
+        <pose>0 -0.06 0 0 0 0</pose>
+        <update_rate>30</update_rate>
+        <always_on>1</always_on>
+        <topic>zed/right</topic>
+        <camera>
+          <image>
+            <format>RGB_INT8</format>
+          </image>
+          <clip>
+            <near>0.01</near>
+            <far>3000</far>
+          </clip>
+        </camera>
+      </sensor>
+  </gazebo>
 </robot>

File: zed_wrapper/urdf/zed_macro.urdf.xacro (robot description, xacro)
@@ -15,5 +15,5 @@
 OF THIS SOFTWARE, EVEN IF ADVISED OF THE POSSIBILITY OF SUCH DAMAGE.
 -->
-<robot xmlns:xacro="http://wiki.ros.org/xacro">
+<robot name="stereolabs_camera" xmlns:xacro="http://wiki.ros.org/xacro">
   <xacro:include filename="$(find zed_wrapper)/urdf/include/materials.urdf.xacro" />
   <xacro:property name="M_PI"     value="3.1415926535897931" />
@@ -25,5 +25,5 @@
       - origin: the xyz/rpy offset from the parent link
   -->
-  <xacro:macro name="zed_camera" params="name=zed model=zed parent mesh_file *origin">
+  <xacro:macro name="zed_camera" params="name=zed model=zed declare_parent=true parent mesh_file *origin">
     <xacro:if value="${model == 'zed'}">
       <xacro:property name="baseline" value="0.12" />
@@ -54,13 +54,23 @@
       <xacro:property name="optical_offset_x" value="-0.01" />
     </xacro:if>
+    <xacro:if value="${declare_parent}">
+      <link name="${parent}" />
+      <joint name="${name}_base_joint" type="fixed">
+        <parent link="${parent}"/>
+        <child link="${name}_base_link"/>
+        <xacro:insert_block name="origin" />
+      </joint>
+    </xacro:if>
     <!-- Camera mounting point (the threaded screw hole in the bottom) -->
-    <link name="${name}_base_link">
+    <link name="${name}_base_link" />
+    <!-- Camera Center -->
+    <link name="${name}_camera_center">
       <visual>
-	      <origin xyz="${screw_offset_x} 0 ${height/2}" rpy="0 0 0"/>
-	      <geometry>
-		      <!-- <mesh filename="package://zed_interfaces/meshes/${model}.stl" /> -->
+        <origin xyz="${screw_offset_x} 0 ${height/2}" rpy="0 0 0"/>
+        <geometry>
+          <!-- <mesh filename="package://zed_interfaces/meshes/${model}.stl" /> -->
           <mesh filename="file://${mesh_file}" />
-	      </geometry>
-	      <material name="${model}_mat" />
+        </geometry>
+        <material name="${model}_mat" />
       </visual>
       <collision>
@@ -75,11 +85,4 @@
       </inertial>
     </link>
-    <joint name="${name}_base_joint" type="fixed">
-      <parent link="${parent}"/>
-      <child link="${name}_base_link"/>
-      <xacro:insert_block name="origin" />
-    </joint>
-    <!-- Camera Center -->
-    <link name="${name}_camera_center" />
     <joint name="${name}_camera_center_joint" type="fixed">
       <parent link="${name}_base_link"/>
