Commit message: Improve ZED xacro/URDF

File: zed_wrapper/urdf/zed_descr.urdf.xacro (robot description, xacro)
@@ -37,6 +37,7 @@
       <zed_serial_number>510</zed_serial_number>
       <zed_resolution>HD720</zed_resolution>
-      <zed_framerate>30</zed_framerate>
+      <zed_framerate>15</zed_framerate>
       <zed_sim_idx>0</zed_sim_idx>
+      <always_on>1</always_on>
     </plugin>
   </gazebo>
@@ -44,5 +45,5 @@
       <sensor name="zed_left" type="camera">
         <pose>0 0.06 0 0 0 0</pose>
-        <update_rate>30</update_rate>
+        <update_rate>15</update_rate>
         <always_on>1</always_on>
         <topic>zed/left</topic>
@@ -53,5 +54,5 @@
           <clip>
             <near>0.01</near>
-            <far>3000</far>
+            <far>300</far>
           </clip>
         </camera>
@@ -59,5 +60,5 @@
       <sensor name="zed_right" type="camera">
         <pose>0 -0.06 0 0 0 0</pose>
-        <update_rate>30</update_rate>
+        <update_rate>15</update_rate>
         <always_on>1</always_on>
         <topic>zed/right</topic>
@@ -68,8 +69,16 @@
           <clip>
             <near>0.01</near>
-            <far>3000</far>
+            <far>300</far>
           </clip>
         </camera>
       </sensor>
   </gazebo>
+  <gazebo>
+    <scene>
+      <ambient>1 1 1 1</ambient>
+      <background>0.3 0.7 0.9 1</background>
+      <shadows>0</shadows>
+      <grid>1</grid>
+    </scene>
+  </gazebo>
 </robot>

File: zed_wrapper/urdf/zed_macro.urdf.xacro (robot description, xacro)
@@ -30,5 +30,5 @@
       <xacro:property name="height" value="0.03" />
       <xacro:property name="bottom_slope" value="0.05" />
-      <xacro:property name="screw_offset_x" value="0.0" />
+      <xacro:property name="screw_offset_x" value="0" />
       <xacro:property name="optical_offset_x" value="-0.01" />
     </xacro:if>
@@ -36,7 +36,7 @@
       <xacro:property name="baseline" value="0.06" />
       <xacro:property name="height" value="0.0265" />
-      <xacro:property name="bottom_slope" value="0.0" />
-      <xacro:property name="screw_offset_x" value="0.0" />
-      <xacro:property name="optical_offset_x" value="0.0" />
+      <xacro:property name="bottom_slope" value="0" />
+      <xacro:property name="screw_offset_x" value="0" />
+      <xacro:property name="optical_offset_x" value="0" />
     </xacro:if>
     <xacro:if value="${model == 'zed2'}">
@@ -44,5 +44,5 @@
       <xacro:property name="height" value="0.03" />
       <xacro:property name="bottom_slope" value="0.05" />
-      <xacro:property name="screw_offset_x" value="0.0" />
+      <xacro:property name="screw_offset_x" value="0" />
       <xacro:property name="optical_offset_x" value="-0.01" />
     </xacro:if>
@@ -50,5 +50,5 @@
       <xacro:property name="baseline" value="0.12" />
       <xacro:property name="height" value="0.03" />
-      <xacro:property name="bottom_slope" value="0.0" />
+      <xacro:property name="bottom_slope" value="0" />
       <xacro:property name="screw_offset_x" value="-0.01" />
       <xacro:property name="optical_offset_x" value="-0.01" />
@@ -63,11 +63,8 @@
     </xacro:if>
     <!-- Camera mounting point (the threaded screw hole in the bottom) -->
-    <link name="${name}_base_link" />
-    <!-- Camera Center -->
-    <link name="${name}_camera_center">
+    <link name="${name}_base_link">
       <visual>
         <origin xyz="${screw_offset_x} 0 ${height/2}" rpy="0 0 0"/>
         <geometry>
-          <!-- <mesh filename="package://zed_interfaces/meshes/${model}.stl" /> -->
           <mesh filename="file://${mesh_file}" />
         </geometry>
@@ -76,13 +73,9 @@
       <collision>
         <geometry>
-          <!-- <mesh filename="package://zed_interfaces/meshes/${model}.stl" /> -->
           <mesh filename="file://${mesh_file}" />
         </geometry>
       </collision>
-      <inertial>
-        <mass value="0.125" />
-        <inertia ixx="0.000028521" ixy="0.0" ixz="0.0" iyy="0.000465434" iyz="0.0" izz="0.000468458"/>
-      </inertial>
     </link>
+    <!-- Camera Center -->
     <joint name="${name}_camera_center_joint" type="fixed">
       <parent link="${name}_base_link"/>
@@ -90,6 +83,11 @@
       <origin xyz="0 0 ${height/2}" rpy="0 ${bottom_slope} 0" />
     </joint>
+    <link name="${name}_camera_center">
+      <inertial>
+        <mass value="0.125" />
+        <inertia ixx="0.000028521" ixy="0" ixz="0" iyy="0.000465434" iyz="0" izz="0.000468458"/>
+      </inertial>
+    </link>
     <!-- Left Camera -->
-    <link name="${name}_left_camera_frame" />
     <joint name="${name}_left_camera_joint" type="fixed">
       <parent link="${name}_camera_center"/>
@@ -97,12 +95,12 @@
       <origin xyz="0 ${baseline/2} 0" rpy="0 0 0" />
     </joint>
-    <link name="${name}_left_camera_optical_frame"/>
+    <link name="${name}_left_camera_frame" />
     <joint name="${name}_left_camera_optical_joint" type="fixed">
-      <origin xyz="${optical_offset_x} 0 0" rpy="-${M_PI/2} 0.0 -${M_PI/2}"/>
+      <origin xyz="${optical_offset_x} 0 0" rpy="-${M_PI/2} 0 -${M_PI/2}"/>
       <parent link="${name}_left_camera_frame"/>
       <child link="${name}_left_camera_optical_frame"/>
     </joint>
+    <link name="${name}_left_camera_optical_frame"/>
     <!-- Right Camera -->
-    <link name="${name}_right_camera_frame" />
     <joint name="${name}_right_camera_joint" type="fixed">
       <parent link="${name}_camera_center"/>
@@ -110,13 +108,13 @@
       <origin xyz="0 -${baseline/2} 0" rpy="0 0 0" />
     </joint>
-    <link name="${name}_right_camera_optical_frame"/>
+    <link name="${name}_right_camera_frame" />
     <joint name="${name}_right_camera_optical_joint" type="fixed">
-      <origin xyz="${optical_offset_x} 0 0" rpy="-${M_PI/2} 0.0 -${M_PI/2}"/>
+      <origin xyz="${optical_offset_x} 0 0" rpy="-${M_PI/2} 0 -${M_PI/2}"/>
       <parent link="${name}_right_camera_frame"/>
       <child link="${name}_right_camera_optical_frame"/>
     </joint>
+    <link name="${name}_right_camera_optical_frame"/>
     <!-- ZED2 Sensors -->
     <xacro:if value="${model == 'zed2' or model == 'zed2i'}">
-      <link name="${name}_mag_link" />
       <joint name="${name}_mag_joint" type="fixed">
         <parent link="${name}_camera_center"/>
@@ -124,5 +122,5 @@
         <origin xyz="0 0 0" rpy="0 0 0" />
       </joint>
-      <link name="${name}_baro_link" />
+      <link name="${name}_mag_link" />
       <joint name="${name}_baro_joint" type="fixed">
         <parent link="${name}_camera_center"/>
@@ -130,5 +128,5 @@
         <origin xyz="0 0 0" rpy="0 0 0" />
       </joint>
-      <link name="${name}_temp_left_link" />
+      <link name="${name}_baro_link" />
       <joint name="${name}_temp_left_joint" type="fixed">
         <parent link="${name}_left_camera_frame"/>
@@ -136,5 +134,5 @@
         <origin xyz="0 0 0" rpy="0 0 0" />
       </joint>
-      <link name="${name}_temp_right_link" />
+      <link name="${name}_temp_left_link" />
       <joint name="${name}_temp_right_joint" type="fixed">
         <parent link="${name}_right_camera_frame"/>
@@ -142,4 +140,5 @@
         <origin xyz="0 0 0" rpy="0 0 0" />
       </joint>
+      <link name="${name}_temp_right_link" />
     </xacro:if>
   </xacro:macro>

Commit message: Removed simulation info from standard URDF

File: zed_wrapper/urdf/zed_descr.urdf.xacro (robot description, xacro)
@@ -15,69 +15,23 @@
 OF THIS SOFTWARE, EVEN IF ADVISED OF THE POSSIBILITY OF SUCH DAMAGE.
 -->
-<robot name="stereolabs_camera" xmlns:xacro="http://ros.org/wiki/xacro">
-  <xacro:arg name="camera_name"     default="zed" />
-  <xacro:arg name="camera_model"    default="zed" />
-  <xacro:arg name="use_base_frame"  default="true" />
-  <xacro:arg name="base_frame"      default="base_link" />
-  <xacro:arg name="cam_pos_x"       default="0.0" />
-  <xacro:arg name="cam_pos_y"       default="0.0" />
-  <xacro:arg name="cam_pos_z"       default="0.0" />
-  <xacro:arg name="cam_roll"        default="0.0" />
-  <xacro:arg name="cam_pitch"       default="0.0" />
-  <xacro:arg name="cam_yaw"         default="0.0" />
-  <xacro:arg name="mesh_file"       default="" />
-  <xacro:include filename="$(find zed_wrapper)/urdf/zed_macro.urdf.xacro" />
-  <xacro:zed_camera name="$(arg camera_name)" model="$(arg camera_model)" declare_parent="$(arg use_base_frame)" parent="$(arg base_frame)" mesh_file="$(arg mesh_file)">
+<robot name="stereolabs_camera_mount" xmlns:xacro="http://ros.org/wiki/xacro">
+	<xacro:arg name="camera_name" default="zed" />
+	<xacro:arg name="camera_model" default="zed" />
+	<xacro:arg name="base_frame" default="base_link" />
+	<xacro:arg name="cam_pos_x" default="0.0" />
+	<xacro:arg name="cam_pos_y" default="0.0" />
+	<xacro:arg name="cam_pos_z" default="0.0" />
+	<xacro:arg name="cam_roll" default="0.0" />
+	<xacro:arg name="cam_pitch" default="0.0" />
+	<xacro:arg name="cam_yaw" default="0.0" />
+  <!-- Robot Base Link-->
+  <link name="$(arg base_frame)" />
+  <!-- Camera Joint-->
+  <joint name="$(arg camera_name)_base_joint" type="fixed">
+    <parent link="$(arg base_frame)"/>
+    <child link="$(arg camera_name)_base_link"/>
     <origin xyz="$(arg cam_pos_x) $(arg cam_pos_y) $(arg cam_pos_z)" rpy="$(arg cam_roll) $(arg cam_pitch) $(arg cam_yaw)" />
-  </xacro:zed_camera>
-  <gazebo>
-    <plugin name="sl_simul::ZedSystem" filename="ZedIgnitionPlugin">
-      <zed_model>zed</zed_model>
-      <zed_serial_number>510</zed_serial_number>
-      <zed_resolution>HD720</zed_resolution>
-      <zed_framerate>15</zed_framerate>
-      <zed_sim_idx>0</zed_sim_idx>
-      <always_on>1</always_on>
-    </plugin>
-  </gazebo>
-  <gazebo reference="$(arg camera_name)_base_link">
-      <sensor name="zed_left" type="camera">
-        <pose>0 0.06 0 0 0 0</pose>
-        <update_rate>15</update_rate>
-        <always_on>1</always_on>
-        <topic>/zed/left</topic>
-        <camera>
-          <image>
-            <format>RGB_INT8</format>
-          </image>
-          <clip>
-            <near>0.01</near>
-            <far>300</far>
-          </clip>
-        </camera>
-      </sensor>
-      <sensor name="zed_right" type="camera">
-        <pose>0 -0.06 0 0 0 0</pose>
-        <update_rate>15</update_rate>
-        <always_on>1</always_on>
-        <topic>/zed/right</topic>
-        <camera>
-          <image>
-            <format>RGB_INT8</format>
-          </image>
-          <clip>
-            <near>0.01</near>
-            <far>300</far>
-          </clip>
-        </camera>
-      </sensor>
-  </gazebo>
-  <gazebo>
-    <scene>
-      <ambient>1 1 1 1</ambient>
-      <background>0.3 0.7 0.9 1</background>
-      <shadows>0</shadows>
-      <grid>1</grid>
-    </scene>
-  </gazebo>
+  </joint>
+	<xacro:include filename="$(find zed_wrapper)/urdf/zed_macro.urdf.xacro" />
+	<xacro:zed_camera name="$(arg camera_name)" model="$(arg camera_model)" parent="$(arg base_frame)" />
 </robot>

File: zed_wrapper/urdf/zed_macro.urdf.xacro (robot description, xacro)
@@ -15,8 +15,8 @@
 OF THIS SOFTWARE, EVEN IF ADVISED OF THE POSSIBILITY OF SUCH DAMAGE.
 -->
-<robot name="stereolabs_camera" xmlns:xacro="http://wiki.ros.org/xacro">
-  <xacro:include filename="$(find zed_wrapper)/urdf/include/materials.urdf.xacro" />
-  <xacro:property name="M_PI"     value="3.1415926535897931" />
-  <!--
+<robot xmlns:xacro="http://wiki.ros.org/xacro">
+	<xacro:include filename="$(find zed_wrapper)/urdf/include/materials.urdf.xacro" />
+	<xacro:property name="M_PI" value="3.1415926535897931" />
+	<!--
     Parameters:
       - name: the camera's name.  should match the parameter sent to the launch file for this camera
@@ -25,121 +25,108 @@
       - origin: the xyz/rpy offset from the parent link
   -->
-  <xacro:macro name="zed_camera" params="name=zed model=zed declare_parent=true parent mesh_file *origin">
-    <xacro:if value="${model == 'zed'}">
-      <xacro:property name="baseline" value="0.12" />
-      <xacro:property name="height" value="0.03" />
-      <xacro:property name="bottom_slope" value="0.05" />
-      <xacro:property name="screw_offset_x" value="0" />
-      <xacro:property name="optical_offset_x" value="-0.01" />
-    </xacro:if>
-    <xacro:if value="${model == 'zedm'}">
-      <xacro:property name="baseline" value="0.06" />
-      <xacro:property name="height" value="0.0265" />
-      <xacro:property name="bottom_slope" value="0" />
-      <xacro:property name="screw_offset_x" value="0" />
-      <xacro:property name="optical_offset_x" value="0" />
-    </xacro:if>
-    <xacro:if value="${model == 'zed2'}">
-      <xacro:property name="baseline" value="0.12" />
-      <xacro:property name="height" value="0.03" />
-      <xacro:property name="bottom_slope" value="0.05" />
-      <xacro:property name="screw_offset_x" value="0" />
-      <xacro:property name="optical_offset_x" value="-0.01" />
-    </xacro:if>
-    <xacro:if value="${model == 'zed2i'}">
-      <xacro:property name="baseline" value="0.12" />
-      <xacro:property name="height" value="0.03" />
-      <xacro:property name="bottom_slope" value="0" />
-      <xacro:property name="screw_offset_x" value="-0.01" />
-      <xacro:property name="optical_offset_x" value="-0.01" />
-    </xacro:if>
-    <xacro:if value="${declare_parent}">
-      <link name="${parent}" />
-      <joint name="${name}_base_joint" type="fixed">
-        <parent link="${parent}"/>
-        <child link="${name}_base_link"/>
-        <xacro:insert_block name="origin" />
-      </joint>
-    </xacro:if>
+	<xacro:macro name="zed_camera" params="name=zed model=zed parent">
+		<xacro:if value="${model == 'zed'}">
+			<xacro:property name="baseline" value="0.12" />
+			<xacro:property name="height" value="0.03" />
+			<xacro:property name="bottom_slope" value="0.05" />
+			<xacro:property name="screw_offset_x" value="0.0" />
+			<xacro:property name="optical_offset_x" value="-0.01" />
+		</xacro:if>
+		<xacro:if value="${model == 'zedm'}">
+			<xacro:property name="baseline" value="0.06" />
+			<xacro:property name="height" value="0.0265" />
+			<xacro:property name="bottom_slope" value="0.0" />
+			<xacro:property name="screw_offset_x" value="0.0" />
+			<xacro:property name="optical_offset_x" value="0.0" />
+		</xacro:if>
+		<xacro:if value="${model == 'zed2'}">
+			<xacro:property name="baseline" value="0.12" />
+			<xacro:property name="height" value="0.03" />
+			<xacro:property name="bottom_slope" value="0.05" />
+			<xacro:property name="screw_offset_x" value="0.0" />
+			<xacro:property name="optical_offset_x" value="-0.01" />
+		</xacro:if>
+		<xacro:if value="${model == 'zed2i'}">
+			<xacro:property name="baseline" value="0.12" />
+			<xacro:property name="height" value="0.03" />
+			<xacro:property name="bottom_slope" value="0.0" />
+			<xacro:property name="screw_offset_x" value="-0.01" />
+			<xacro:property name="optical_offset_x" value="-0.01" />
+		</xacro:if>
     <!-- Camera mounting point (the threaded screw hole in the bottom) -->
-    <link name="${name}_base_link">
-      <visual>
-        <origin xyz="${screw_offset_x} 0 ${height/2}" rpy="0 0 0"/>
-        <geometry>
-          <mesh filename="file://${mesh_file}" />
-        </geometry>
-        <material name="${model}_mat" />
-      </visual>
-      <collision>
-        <geometry>
-          <mesh filename="file://${mesh_file}" />
-        </geometry>
-      </collision>
-    </link>
-    <!-- Camera Center -->
-    <joint name="${name}_camera_center_joint" type="fixed">
-      <parent link="${name}_base_link"/>
-      <child link="${name}_camera_center"/>
-      <origin xyz="0 0 ${height/2}" rpy="0 ${bottom_slope} 0" />
-    </joint>
-    <link name="${name}_camera_center">
-      <inertial>
-        <mass value="0.125" />
-        <inertia ixx="0.000028521" ixy="0" ixz="0" iyy="0.000465434" iyz="0" izz="0.000468458"/>
-      </inertial>
-    </link>
-    <!-- Left Camera -->
-    <joint name="${name}_left_camera_joint" type="fixed">
-      <parent link="${name}_camera_center"/>
-      <child link="${name}_left_camera_frame"/>
-      <origin xyz="0 ${baseline/2} 0" rpy="0 0 0" />
-    </joint>
-    <link name="${name}_left_camera_frame" />
-    <joint name="${name}_left_camera_optical_joint" type="fixed">
-      <origin xyz="${optical_offset_x} 0 0" rpy="-${M_PI/2} 0 -${M_PI/2}"/>
-      <parent link="${name}_left_camera_frame"/>
-      <child link="${name}_left_camera_optical_frame"/>
-    </joint>
-    <link name="${name}_left_camera_optical_frame"/>
-    <!-- Right Camera -->
-    <joint name="${name}_right_camera_joint" type="fixed">
-      <parent link="${name}_camera_center"/>
-      <child link="${name}_right_camera_frame"/>
-      <origin xyz="0 -${baseline/2} 0" rpy="0 0 0" />
-    </joint>
-    <link name="${name}_right_camera_frame" />
-    <joint name="${name}_right_camera_optical_joint" type="fixed">
-      <origin xyz="${optical_offset_x} 0 0" rpy="-${M_PI/2} 0 -${M_PI/2}"/>
-      <parent link="${name}_right_camera_frame"/>
-      <child link="${name}_right_camera_optical_frame"/>
-    </joint>
-    <link name="${name}_right_camera_optical_frame"/>
-    <!-- ZED2 Sensors -->
-    <xacro:if value="${model == 'zed2' or model == 'zed2i'}">
-      <joint name="${name}_mag_joint" type="fixed">
-        <parent link="${name}_camera_center"/>
-        <child link="${name}_mag_link"/>
-        <origin xyz="0 0 0" rpy="0 0 0" />
-      </joint>
-      <link name="${name}_mag_link" />
-      <joint name="${name}_baro_joint" type="fixed">
-        <parent link="${name}_camera_center"/>
-        <child link="${name}_baro_link"/>
-        <origin xyz="0 0 0" rpy="0 0 0" />
-      </joint>
-      <link name="${name}_baro_link" />
-      <joint name="${name}_temp_left_joint" type="fixed">
-        <parent link="${name}_left_camera_frame"/>
-        <child link="${name}_temp_left_link"/>
-        <origin xyz="0 0 0" rpy="0 0 0" />
-      </joint>
-      <link name="${name}_temp_left_link" />
-      <joint name="${name}_temp_right_joint" type="fixed">
-        <parent link="${name}_right_camera_frame"/>
-        <child link="${name}_temp_right_link"/>
-        <origin xyz="0 0 0" rpy="0 0 0" />
-      </joint>
-      <link name="${name}_temp_right_link" />
-    </xacro:if>
-  </xacro:macro>
+    <link name="${name}_base_link" />
+		<!-- Camera Center -->
+		<link name="${name}_camera_center">
+			<visual>
+				<origin xyz="${screw_offset_x} 0 0" rpy="0 0 0"/>
+				<geometry>
+					<mesh filename="package://zed_interfaces/meshes/${model}.stl" />
+				</geometry>
+				<material name="${model}_mat" />
+			</visual>
+			<collision>
+				<geometry>
+					<mesh filename="package://zed_interfaces/meshes/${model}.stl" />
+				</geometry>
+			</collision>
+		</link>
+		<joint name="${name}_camera_center_joint" type="fixed">
+			<parent link="${name}_base_link"/>
+			<child link="${name}_camera_center"/>
+			<origin xyz="0 0 ${height/2}" rpy="0 ${bottom_slope} 0" />
+		</joint>
+		<!-- Left Camera -->
+		<link name="${name}_left_camera_frame" />
+		<joint name="${name}_left_camera_joint" type="fixed">
+			<parent link="${name}_camera_center"/>
+			<child link="${name}_left_camera_frame"/>
+			<origin xyz="0 ${baseline/2} 0" rpy="0 0 0" />
+		</joint>
+		<link name="${name}_left_camera_optical_frame"/>
+		<joint name="${name}_left_camera_optical_joint" type="fixed">
+			<origin xyz="${optical_offset_x} 0 0" rpy="-${M_PI/2} 0.0 -${M_PI/2}"/>
+			<parent link="${name}_left_camera_frame"/>
+			<child link="${name}_left_camera_optical_frame"/>
+		</joint>
+		<!-- Right Camera -->
+		<link name="${name}_right_camera_frame" />
+		<joint name="${name}_right_camera_joint" type="fixed">
+			<parent link="${name}_camera_center"/>
+			<child link="${name}_right_camera_frame"/>
+			<origin xyz="0 -${baseline/2} 0" rpy="0 0 0" />
+		</joint>
+		<link name="${name}_right_camera_optical_frame"/>
+		<joint name="${name}_right_camera_optical_joint" type="fixed">
+			<origin xyz="${optical_offset_x} 0 0" rpy="-${M_PI/2} 0.0 -${M_PI/2}"/>
+			<parent link="${name}_right_camera_frame"/>
+			<child link="${name}_right_camera_optical_frame"/>
+		</joint>
+		<!-- ZED2 Sensors -->
+		<xacro:if value="${model == 'zed2' or model == 'zed2i'}">
+			<link name="${name}_mag_link" />
+			<joint name="${name}_mag_joint" type="fixed">
+				<parent link="${name}_camera_center"/>
+				<child link="${name}_mag_link"/>
+				<origin xyz="0 0 0" rpy="0 0 0" />
+			</joint>
+			<link name="${name}_baro_link" />
+			<joint name="${name}_baro_joint" type="fixed">
+				<parent link="${name}_camera_center"/>
+				<child link="${name}_baro_link"/>
+				<origin xyz="0 0 0" rpy="0 0 0" />
+			</joint>
+			<link name="${name}_temp_left_link" />
+			<joint name="${name}_temp_left_joint" type="fixed">
+				<parent link="${name}_left_camera_frame"/>
+				<child link="${name}_temp_left_link"/>
+				<origin xyz="0 0 0" rpy="0 0 0" />
+			</joint>
+			<link name="${name}_temp_right_link" />
+			<joint name="${name}_temp_right_joint" type="fixed">
+				<parent link="${name}_right_camera_frame"/>
+				<child link="${name}_temp_right_link"/>
+				<origin xyz="0 0 0" rpy="0 0 0" />
+			</joint>
+		</xacro:if>
+	</xacro:macro>
 </robot>
