Commit message: Fix URDF/Xacro

File: zed_wrapper/urdf/zed_descr.urdf.xacro (robot description, xacro)
@@ -25,7 +25,8 @@
 	<xacro:arg name="cam_pitch" default="0.0" />
 	<xacro:arg name="cam_yaw" default="0.0" />
+  <xacro:arg name="mesh_file" default="" />
   <!-- Robot Base Link-->
   <link name="$(arg base_frame)" />
-  <!-- Camera Joint-->
+  <!-- Camera Base Joint-->
   <joint name="$(arg camera_name)_base_joint" type="fixed">
     <parent link="$(arg base_frame)"/>
@@ -34,4 +35,4 @@
   </joint>
 	<xacro:include filename="$(find zed_wrapper)/urdf/zed_macro.urdf.xacro" />
-	<xacro:zed_camera name="$(arg camera_name)" model="$(arg camera_model)" parent="$(arg base_frame)" />
+	<xacro:zed_camera name="$(arg camera_name)" model="$(arg camera_model)" parent="$(arg base_frame)" mesh_file="$(arg mesh_file)" />
 </robot>

File: zed_wrapper/urdf/zed_macro.urdf.xacro (robot description, xacro)
@@ -25,5 +25,5 @@
       - origin: the xyz/rpy offset from the parent link
   -->
-	<xacro:macro name="zed_camera" params="name=zed model=zed parent">
+	<xacro:macro name="zed_camera" params="name=zed model=zed parent mesh_file">
 		<xacro:if value="${model == 'zed'}">
 			<xacro:property name="baseline" value="0.12" />
@@ -66,13 +66,17 @@
 				<origin xyz="${screw_offset_x} 0 0" rpy="0 0 0"/>
 				<geometry>
-					<mesh filename="package://zed_interfaces/meshes/${model}.stl" />
-				</geometry>
+					<mesh filename="file://${mesh_file}" />
+        </geometry>
 				<material name="${model}_mat" />
 			</visual>
 			<collision>
 				<geometry>
-					<mesh filename="package://zed_interfaces/meshes/${model}.stl" />
+					<mesh filename="file://${mesh_file}" />
 				</geometry>
 			</collision>
+      <inertial>
+        <mass value="0.125" />
+        <inertia ixx="0.000028521" ixy="0.0" ixz="0.0" iyy="0.000465434" iyz="0.0" izz="0.000468458"/>
+      </inertial>
 		</link>
 		<!-- Left Camera -->
@@ -102,5 +106,5 @@
     </joint>
 		<link name="${name}_right_camera_optical_frame"/>
-		<!-- ZED2 Sensors -->
+		<!-- Sensors -->
 		<xacro:if value="${model == 'zed2' or model == 'zed2i'}">
       <joint name="${name}_mag_joint" type="fixed">

Commit message: Fixes for simulation

File: zed_wrapper/urdf/zed_descr.urdf.xacro (robot description, xacro)
@@ -26,13 +26,13 @@
 	<xacro:arg name="cam_yaw" default="0.0" />
 	<xacro:arg name="mesh_file" default="" />
-	<!-- Robot Base Link-->
+	<!-- Robot Base link -->
 	<link name="$(arg base_frame)" />
-	<!-- Camera Base Joint-->
-	<joint name="$(arg camera_name)_base_joint" type="fixed">
-		<parent link="$(arg base_frame)"/>
-		<child link="$(arg camera_name)_base_link"/>
+	<!-- ZED mount -->
+	<xacro:include filename="$(find zed_wrapper)/urdf/zed_mount_macro.urdf.xacro" />
+	<xacro:zed_mount cam_name="$(arg camera_name)" parent="$(arg base_frame)">
 		<origin xyz="$(arg cam_pos_x) $(arg cam_pos_y) $(arg cam_pos_z)" rpy="$(arg cam_roll) $(arg cam_pitch) $(arg cam_yaw)" />
-	</joint>
+	</xacro:zed_mount>
+	<!-- ZED -->
 	<xacro:include filename="$(find zed_wrapper)/urdf/zed_macro.urdf.xacro" />
-	<xacro:zed_camera name="$(arg camera_name)" model="$(arg camera_model)" parent="$(arg base_frame)" mesh_file="$(arg mesh_file)" />
+	<xacro:zed_camera cam_name="$(arg camera_name)" model="$(arg camera_model)" parent="$(arg base_frame)" mesh_file="$(arg mesh_file)" />
 </robot>

File: zed_wrapper/urdf/zed_macro.urdf.xacro (robot description, xacro)
@@ -20,10 +20,10 @@
 	<!--
     Parameters:
-      - name: the camera's name.  should match the parameter sent to the launch file for this camera
+      - cam_name: the camera's name.  should match the parameter sent to the launch file for this camera
       - model: the tye of camera, one of zed, zedm, zed2, zed2i
       - parent: [REQUIRED] the parent link of the camera.  must be defined in the URDF file that uses this macro
       - mesh_file: [REQUIRED] the file containing the 3D model of the camera
   -->
-	<xacro:macro name="zed_camera" params="name=zed model=zed parent mesh_file">
+	<xacro:macro name="zed_camera" params="cam_name=zed model=zed parent mesh_file">
 		<xacro:if value="${model == 'zed'}">
 			<xacro:property name="baseline" value="0.12" />
@@ -55,12 +55,12 @@
 		</xacro:if>
 		<!-- Camera mounting point (the threaded screw hole in the bottom) -->
-		<link name="${name}_base_link" />
+		<link name="${cam_name}_base_link" />
 		<!-- Camera Center -->
-		<joint name="${name}_camera_center_joint" type="fixed">
-			<parent link="${name}_base_link"/>
-			<child link="${name}_camera_center"/>
+		<joint name="${cam_name}_camera_center_joint" type="fixed">
+			<parent link="${cam_name}_base_link"/>
+			<child link="${cam_name}_camera_center"/>
 			<origin xyz="0 0 ${height/2}" rpy="0 ${bottom_slope} 0" />
 		</joint>
-		<link name="${name}_camera_center">
+		<link name="${cam_name}_camera_center">
 			<visual>
 				<origin xyz="${screw_offset_x} 0 0" rpy="0 0 0"/>
@@ -81,55 +81,55 @@
 		</link>
 		<!-- Left Camera -->
-		<joint name="${name}_left_camera_joint" type="fixed">
-			<parent link="${name}_camera_center"/>
-			<child link="${name}_left_camera_frame"/>
+		<joint name="${cam_name}_left_camera_joint" type="fixed">
+			<parent link="${cam_name}_camera_center"/>
+			<child link="${cam_name}_left_camera_frame"/>
 			<origin xyz="0 ${baseline/2} 0" rpy="0 0 0" />
 		</joint>
-		<link name="${name}_left_camera_frame" />
-		<joint name="${name}_left_camera_optical_joint" type="fixed">
+		<link name="${cam_name}_left_camera_frame" />
+		<joint name="${cam_name}_left_camera_optical_joint" type="fixed">
 			<origin xyz="${optical_offset_x} 0 0" rpy="-${M_PI/2} 0.0 -${M_PI/2}"/>
-			<parent link="${name}_left_camera_frame"/>
-			<child link="${name}_left_camera_optical_frame"/>
+			<parent link="${cam_name}_left_camera_frame"/>
+			<child link="${cam_name}_left_camera_optical_frame"/>
 		</joint>
-		<link name="${name}_left_camera_optical_frame"/>
+		<link name="${cam_name}_left_camera_optical_frame"/>
 		<!-- Right Camera -->
-		<joint name="${name}_right_camera_joint" type="fixed">
-			<parent link="${name}_camera_center"/>
-			<child link="${name}_right_camera_frame"/>
+		<joint name="${cam_name}_right_camera_joint" type="fixed">
+			<parent link="${cam_name}_camera_center"/>
+			<child link="${cam_name}_right_camera_frame"/>
 			<origin xyz="0 -${baseline/2} 0" rpy="0 0 0" />
 		</joint>
-		<link name="${name}_right_camera_frame" />
-		<joint name="${name}_right_camera_optical_joint" type="fixed">
+		<link name="${cam_name}_right_camera_frame" />
+		<joint name="${cam_name}_right_camera_optical_joint" type="fixed">
 			<origin xyz="${optical_offset_x} 0 0" rpy="-${M_PI/2} 0.0 -${M_PI/2}"/>
-			<parent link="${name}_right_camera_frame"/>
-			<child link="${name}_right_camera_optical_frame"/>
+			<parent link="${cam_name}_right_camera_frame"/>
+			<child link="${cam_name}_right_camera_optical_frame"/>
 		</joint>
-		<link name="${name}_right_camera_optical_frame"/>
+		<link name="${cam_name}_right_camera_optical_frame"/>
 		<!-- Sensors -->
 		<xacro:if value="${model == 'zed2' or model == 'zed2i'}">
-			<joint name="${name}_mag_joint" type="fixed">
-				<parent link="${name}_camera_center"/>
-				<child link="${name}_mag_link"/>
+			<joint name="${cam_name}_mag_joint" type="fixed">
+				<parent link="${cam_name}_camera_center"/>
+				<child link="${cam_name}_mag_link"/>
 				<origin xyz="0 0 0" rpy="0 0 0" />
 			</joint>
-			<link name="${name}_mag_link" />
-			<joint name="${name}_baro_joint" type="fixed">
-				<parent link="${name}_camera_center"/>
-				<child link="${name}_baro_link"/>
+			<link name="${cam_name}_mag_link" />
+			<joint name="${cam_name}_baro_joint" type="fixed">
+				<parent link="${cam_name}_camera_center"/>
+				<child link="${cam_name}_baro_link"/>
 				<origin xyz="0 0 0" rpy="0 0 0" />
 			</joint>
-			<link name="${name}_baro_link" />
-			<joint name="${name}_temp_left_joint" type="fixed">
-				<parent link="${name}_left_camera_frame"/>
-				<child link="${name}_temp_left_link"/>
+			<link name="${cam_name}_baro_link" />
+			<joint name="${cam_name}_temp_left_joint" type="fixed">
+				<parent link="${cam_name}_left_camera_frame"/>
+				<child link="${cam_name}_temp_left_link"/>
 				<origin xyz="0 0 0" rpy="0 0 0" />
 			</joint>
-			<link name="${name}_temp_left_link" />
-			<joint name="${name}_temp_right_joint" type="fixed">
-				<parent link="${name}_right_camera_frame"/>
-				<child link="${name}_temp_right_link"/>
+			<link name="${cam_name}_temp_left_link" />
+			<joint name="${cam_name}_temp_right_joint" type="fixed">
+				<parent link="${cam_name}_right_camera_frame"/>
+				<child link="${cam_name}_temp_right_link"/>
 				<origin xyz="0 0 0" rpy="0 0 0" />
 			</joint>
-			<link name="${name}_temp_right_link" />
+			<link name="${cam_name}_temp_right_link" />
 		</xacro:if>
 	</xacro:macro>
