Commit message: Fix copyright and minor fixes

File: zed_wrapper/urdf/include/materials.urdf.xacro (robot description, xacro)
@@ -1,5 +1,5 @@
 <?xml version="1.0"?>
 <!--
-Copyright (c) 2020, STEREOLABS.
+Copyright (c) 2022, STEREOLABS.
 All rights reserved.
 THIS SOFTWARE IS PROVIDED BY THE COPYRIGHT HOLDERS AND CONTRIBUTORS
@@ -16,15 +16,15 @@
 -->
 <robot>
-    <material name="zed_mat">
-        <color rgba="0.8 0.8 0.8 1.0"/>
-    </material>
-    <material name="zedm_mat">
-        <color rgba="0 0 0 1.0"/>
-    </material>
-    <material name="zed2_mat">
-        <color rgba="0.25 0.25 0.25 1.0"/>
-    </material>
-    <material name="zed2i_mat">
-        <color rgba="0.25 0.25 0.25 1.0"/>
-    </material>
+	<material name="zed_mat">
+		<color rgba="0.8 0.8 0.8 1.0"/>
+	</material>
+	<material name="zedm_mat">
+		<color rgba="0 0 0 1.0"/>
+	</material>
+	<material name="zed2_mat">
+		<color rgba="0.25 0.25 0.25 1.0"/>
+	</material>
+	<material name="zed2i_mat">
+		<color rgba="0.25 0.25 0.25 1.0"/>
+	</material>
 </robot>

File: zed_wrapper/urdf/zed_descr.urdf.xacro (robot description, xacro)
@@ -1,5 +1,5 @@
 <?xml version="1.0"?>
 <!--
-Copyright (c) 2020, STEREOLABS.
+Copyright (c) 2022, STEREOLABS.
 All rights reserved.
 THIS SOFTWARE IS PROVIDED BY THE COPYRIGHT HOLDERS AND CONTRIBUTORS
@@ -25,13 +25,13 @@
 	<xacro:arg name="cam_pitch" default="0.0" />
 	<xacro:arg name="cam_yaw" default="0.0" />
-  <xacro:arg name="mesh_file" default="" />
-  <!-- Robot Base Link-->
-  <link name="$(arg base_frame)" />
-  <!-- Camera Base Joint-->
-  <joint name="$(arg camera_name)_base_joint" type="fixed">
-    <parent link="$(arg base_frame)"/>
-    <child link="$(arg camera_name)_base_link"/>
-    <origin xyz="$(arg cam_pos_x) $(arg cam_pos_y) $(arg cam_pos_z)" rpy="$(arg cam_roll) $(arg cam_pitch) $(arg cam_yaw)" />
-  </joint>
+	<xacro:arg name="mesh_file" default="" />
+	<!-- Robot Base Link-->
+	<link name="$(arg base_frame)" />
+	<!-- Camera Base Joint-->
+	<joint name="$(arg camera_name)_base_joint" type="fixed">
+		<parent link="$(arg base_frame)"/>
+		<child link="$(arg camera_name)_base_link"/>
+		<origin xyz="$(arg cam_pos_x) $(arg cam_pos_y) $(arg cam_pos_z)" rpy="$(arg cam_roll) $(arg cam_pitch) $(arg cam_yaw)" />
+	</joint>
 	<xacro:include filename="$(find zed_wrapper)/urdf/zed_macro.urdf.xacro" />
 	<xacro:zed_camera name="$(arg camera_name)" model="$(arg camera_model)" parent="$(arg base_frame)" mesh_file="$(arg mesh_file)" />

File: zed_wrapper/urdf/zed_macro.urdf.xacro (robot description, xacro)
@@ -1,5 +1,5 @@
 <?xml version="1.0"?>
 <!--
-Copyright (c) 2020, STEREOLABS.
+Copyright (c) 2022, STEREOLABS.
 All rights reserved.
 THIS SOFTWARE IS PROVIDED BY THE COPYRIGHT HOLDERS AND CONTRIBUTORS
@@ -54,12 +54,12 @@
 			<xacro:property name="optical_offset_x" value="-0.01" />
 		</xacro:if>
-    <!-- Camera mounting point (the threaded screw hole in the bottom) -->
-    <link name="${name}_base_link" />
+		<!-- Camera mounting point (the threaded screw hole in the bottom) -->
+		<link name="${name}_base_link" />
 		<!-- Camera Center -->
-    <joint name="${name}_camera_center_joint" type="fixed">
-      <parent link="${name}_base_link"/>
-      <child link="${name}_camera_center"/>
-      <origin xyz="0 0 ${height/2}" rpy="0 ${bottom_slope} 0" />
-    </joint>
+		<joint name="${name}_camera_center_joint" type="fixed">
+			<parent link="${name}_base_link"/>
+			<child link="${name}_camera_center"/>
+			<origin xyz="0 0 ${height/2}" rpy="0 ${bottom_slope} 0" />
+		</joint>
 		<link name="${name}_camera_center">
 			<visual>
@@ -67,5 +67,5 @@
 				<geometry>
 					<mesh filename="file://${mesh_file}" />
-        </geometry>
+				</geometry>
 				<material name="${model}_mat" />
 			</visual>
@@ -75,60 +75,60 @@
 				</geometry>
 			</collision>
-      <inertial>
-        <mass value="0.125" />
-        <inertia ixx="0.000028521" ixy="0.0" ixz="0.0" iyy="0.000465434" iyz="0.0" izz="0.000468458"/>
-      </inertial>
+			<inertial>
+				<mass value="0.125" />
+				<inertia ixx="0.000028521" ixy="0.0" ixz="0.0" iyy="0.000465434" iyz="0.0" izz="0.000468458"/>
+			</inertial>
 		</link>
 		<!-- Left Camera -->
-    <joint name="${name}_left_camera_joint" type="fixed">
-      <parent link="${name}_camera_center"/>
-      <child link="${name}_left_camera_frame"/>
-      <origin xyz="0 ${baseline/2} 0" rpy="0 0 0" />
-    </joint>
+		<joint name="${name}_left_camera_joint" type="fixed">
+			<parent link="${name}_camera_center"/>
+			<child link="${name}_left_camera_frame"/>
+			<origin xyz="0 ${baseline/2} 0" rpy="0 0 0" />
+		</joint>
 		<link name="${name}_left_camera_frame" />
-    <joint name="${name}_left_camera_optical_joint" type="fixed">
-      <origin xyz="${optical_offset_x} 0 0" rpy="-${M_PI/2} 0.0 -${M_PI/2}"/>
-      <parent link="${name}_left_camera_frame"/>
-      <child link="${name}_left_camera_optical_frame"/>
-    </joint>
+		<joint name="${name}_left_camera_optical_joint" type="fixed">
+			<origin xyz="${optical_offset_x} 0 0" rpy="-${M_PI/2} 0.0 -${M_PI/2}"/>
+			<parent link="${name}_left_camera_frame"/>
+			<child link="${name}_left_camera_optical_frame"/>
+		</joint>
 		<link name="${name}_left_camera_optical_frame"/>
 		<!-- Right Camera -->
-    <joint name="${name}_right_camera_joint" type="fixed">
-      <parent link="${name}_camera_center"/>
-      <child link="${name}_right_camera_frame"/>
-      <origin xyz="0 -${baseline/2} 0" rpy="0 0 0" />
-    </joint>
+		<joint name="${name}_right_camera_joint" type="fixed">
+			<parent link="${name}_camera_center"/>
+			<child link="${name}_right_camera_frame"/>
+			<origin xyz="0 -${baseline/2} 0" rpy="0 0 0" />
+		</joint>
 		<link name="${name}_right_camera_frame" />
-    <joint name="${name}_right_camera_optical_joint" type="fixed">
-      <origin xyz="${optical_offset_x} 0 0" rpy="-${M_PI/2} 0.0 -${M_PI/2}"/>
-      <parent link="${name}_right_camera_frame"/>
-      <child link="${name}_right_camera_optical_frame"/>
-    </joint>
+		<joint name="${name}_right_camera_optical_joint" type="fixed">
+			<origin xyz="${optical_offset_x} 0 0" rpy="-${M_PI/2} 0.0 -${M_PI/2}"/>
+			<parent link="${name}_right_camera_frame"/>
+			<child link="${name}_right_camera_optical_frame"/>
+		</joint>
 		<link name="${name}_right_camera_optical_frame"/>
 		<!-- Sensors -->
 		<xacro:if value="${model == 'zed2' or model == 'zed2i'}">
-      <joint name="${name}_mag_joint" type="fixed">
-        <parent link="${name}_camera_center"/>
-        <child link="${name}_mag_link"/>
-        <origin xyz="0 0 0" rpy="0 0 0" />
-      </joint>
+			<joint name="${name}_mag_joint" type="fixed">
+				<parent link="${name}_camera_center"/>
+				<child link="${name}_mag_link"/>
+				<origin xyz="0 0 0" rpy="0 0 0" />
+			</joint>
 			<link name="${name}_mag_link" />
-      <joint name="${name}_baro_joint" type="fixed">
-        <parent link="${name}_camera_center"/>
-        <child link="${name}_baro_link"/>
-        <origin xyz="0 0 0" rpy="0 0 0" />
-      </joint>
+			<joint name="${name}_baro_joint" type="fixed">
+				<parent link="${name}_camera_center"/>
+				<child link="${name}_baro_link"/>
+				<origin xyz="0 0 0" rpy="0 0 0" />
+			</joint>
 			<link name="${name}_baro_link" />
-      <joint name="${name}_temp_left_joint" type="fixed">
-        <parent link="${name}_left_camera_frame"/>
-        <child link="${name}_temp_left_link"/>
-        <origin xyz="0 0 0" rpy="0 0 0" />
-      </joint>
+			<joint name="${name}_temp_left_joint" type="fixed">
+				<parent link="${name}_left_camera_frame"/>
+				<child link="${name}_temp_left_link"/>
+				<origin xyz="0 0 0" rpy="0 0 0" />
+			</joint>
 			<link name="${name}_temp_left_link" />
-      <joint name="${name}_temp_right_joint" type="fixed">
-        <parent link="${name}_right_camera_frame"/>
-        <child link="${name}_temp_right_link"/>
-        <origin xyz="0 0 0" rpy="0 0 0" />
-      </joint>
+			<joint name="${name}_temp_right_joint" type="fixed">
+				<parent link="${name}_right_camera_frame"/>
+				<child link="${name}_temp_right_link"/>
+				<origin xyz="0 0 0" rpy="0 0 0" />
+			</joint>
 			<link name="${name}_temp_right_link" />
 		</xacro:if>
